File: Hardware/GNSS_Splitter.brd (EAGLE design)
At the start: 25.4 x 25.4 mm, 25 parts, among them J1 QWIIC_RIGHT_ANGLE, U1 BP2G1+_POWER_SPLITTER

Commit message: Updates
Parts:
- added ILIM: JUMPER-SMT_2_NO_SILK, SparkFun-Jumpers:SMT-JUMPER_2_NO_SILK
- added U$10: (no value), output:#GND#1
- added U$11: (no value), output:#VIN#0
- added U$12: (no value), output:#VIN#1
- added U$13, U$16: (no value), output:GNSS0
- added U$14, U$18: (no value), output:P0
- added U$15, U$17: (no value), output:S__LITTER0
- added U$19: (no value), output:#ILIM#0
- added U$3, U$7: (no value), output:10
- added U$4, U$8: (no value), output:20
- added U$5, U$6: (no value), output:S0
- added U$9: (no value), output:#GND#0
- moved U$2 8.89 mm to (12.7, 11.4)
- moved LOGO1 4.58 mm to (21.6, 17.8)
- moved R1 0.51 mm to (7.11, 16.1)
Connections:
- net N$2: now also ILIM.2
- net VIN: now also ILIM.1
Routing:
- net VIN: track 23.5 -> 26.1 mm, vias 2 -> 3
- net N$2: track 3.16 -> 5.22 mm, vias 0 -> 1
Changed lines of the file:
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@@
 </element>
 <element name="U$1" library="SparkX" package="SPARKX-SMALL" value="SPARKX-LOGO3" x="21.59" y="17.78" smashed="yes"/>
-<element name="U$2" library="SparkX" package="SPARKX-SMALL" value="SPARKX-LOGO3" x="12.7" y="2.54" smashed="yes" rot="MR0"/>
+<element name="U$2" library="SparkX" package="SPARKX-SMALL" value="SPARKX-LOGO3" x="12.7" y="11.43" smashed="yes" rot="MR0"/>
 <element name="J2" library="SparkFun-Connectors" package="1X02_NO_SILK" value="" x="24.13" y="11.43" smashed="yes" rot="R90">
 <attribute name="NAME" x="22.733" y="10.16" size="0.6096" layer="25" font="vector" ratio="20" rot="R90"/>
@@
 <attribute name="VALUE" x="9.271" y="17.018" size="0.6096" layer="27" font="vector" ratio="20" rot="R270" align="top-center"/>
 </element>
-<element name="R1" library="SparkFun-Resistors" package="0603" value="10" x="7.62" y="16.129" smashed="yes" rot="R180">
-<attribute name="NAME" x="7.62" y="15.367" size="0.6096" layer="25" font="vector" ratio="20" rot="R180" align="bottom-center"/>
-<attribute name="PROD_ID" value="RES-12581" x="7.62" y="8.509" size="1.778" layer="27" ratio="15" rot="R180" display="off"/>
-<attribute name="VALUE" x="7.62" y="16.891" size="0.6096" layer="27" font="vector" ratio="20" rot="R180" align="top-center"/>
+<element name="R1" library="SparkFun-Resistors" package="0603" value="10" x="7.112" y="16.129" smashed="yes" rot="R180">
+<attribute name="NAME" x="7.112" y="15.367" size="0.6096" layer="25" font="vector" ratio="20" rot="R180" align="bottom-center"/>
+<attribute name="PROD_ID" value="RES-12581" x="7.112" y="8.509" size="1.778" layer="27" ratio="15" rot="R180" display="off"/>
+<attribute name="VALUE" x="7.112" y="16.891" size="0.6096" layer="27" font="vector" ratio="20" rot="R180" align="top-center"/>
 </element>
 <element name="FB1" library="SparkFun-Coils" package="0603" value="30Ω/1.8A" x="12.446" y="16.129" smashed="yes">
@@
 <attribute name="VALUE" x="8.889996875" y="6.096" size="0.6096" layer="27" font="vector" ratio="20" rot="SR0" align="top-center"/>
 </element>
-<element name="LOGO1" library="SparkFun-Aesthetics" package="OSHW-LOGO-S" value="OSHW-LOGOS" x="19.05" y="21.59" smashed="yes" rot="MR0"/>
+<element name="LOGO1" library="SparkFun-Aesthetics" package="OSHW-LOGO-S" value="OSHW-LOGOS" x="21.59" y="17.78" smashed="yes" rot="MR0"/>
 <element name="LOGO2" library="SparkFun-Aesthetics" package="QWIIC_6MM" value="QWIIC_LOGO_6MM" x="3.302" y="17.78" smashed="yes"/>
 <element name="FD1" library="SparkFun-Aesthetics" package="FIDUCIAL-1X2" value="FIDUCIAL1X2" x="1.27" y="20.32" smashed="yes" rot="MR0"/>
@@
 <attribute name="VALUE" x="2.54" y="20.828" size="0.6096" layer="27" font="vector" ratio="20" align="top-center"/>
 </element>
+<element name="ILIM" library="SparkFun-Jumpers" package="SMT-JUMPER_2_NO_SILK" package3d_urn="urn:adsk.eagle:package:39279/1" value="JUMPER-SMT_2_NO_SILK" x="7.112" y="16.129" smashed="yes" rot="MR180">
+<attribute name="NAME" x="7.112" y="14.986" size="0.6096" layer="26" font="vector" ratio="20" rot="MR180" align="bottom-center"/>
+<attribute name="VALUE" x="7.112" y="17.272" size="0.6096" layer="28" font="vector" ratio="20" rot="MR180" align="top-center"/>
+</element>
+<element name="U$3" library="output" package="10" value="" x="18.288" y="8.89" smashed="yes"/>
+<element name="U$4" library="output" package="20" value="" x="6.858" y="8.89" smashed="yes"/>
+<element name="U$5" library="output" package="S0" value="" x="11.684" y="18.034" smashed="yes"/>
+<element name="U$6" library="output" package="S0" value="" x="12.7" y="17.78" smashed="yes" rot="MR0"/>
+<element name="U$7" library="output" package="10" value="" x="18.415" y="8.89" smashed="yes" rot="MR0"/>
+<element name="U$8" library="output" package="20" value="" x="6.477" y="8.89" smashed="yes" rot="MR0"/>
+<element name="U$9" library="output" package="#GND#0" value="" x="23.241" y="13.97" smashed="yes"/>
+<element name="U$10" library="output" package="#GND#1" value="" x="23.241" y="13.97" smashed="yes" rot="MR0"/>
+<element name="U$11" library="output" package="#VIN#0" value="" x="23.241" y="11.43" smashed="yes"/>
+<element name="U$12" library="output" package="#VIN#1" value="" x="23.241" y="11.43" smashed="yes" rot="MR0"/>
+<element name="U$13" library="output" package="GNSS0" value="" x="12.7" y="3.81" smashed="yes"/>
+<element name="U$15" library="output" package="S__LITTER0" value="" x="12.7" y="2.54" smashed="yes"/>
+<element name="U$14" library="output" package="P0" value="" x="11.049" y="2.286" smashed="yes"/>
+<element name="U$16" library="output" package="GNSS0" value="" x="12.7" y="3.81" smashed="yes" rot="MR0"/>
+<element name="U$17" library="output" package="S__LITTER0" value="" x="12.7" y="2.54" smashed="yes" rot="MR0"/>
+<element name="U$18" library="output" package="P0" value="" x="14.351" y="2.286" smashed="yes" rot="MR0"/>
+<element name="U$19" library="output" package="#ILIM#0" value="" x="7.112" y="17.907" smashed="yes" rot="MR0"/>
 </elements>
 <signals>
@@
 <via x="21.59" y="10.16" extent="1-16" drill="0.3"/>
 <via x="3.81" y="11.43" extent="1-16" drill="0.3"/>
-<via x="6.35" y="8.89" extent="1-16" drill="0.3"/>
 <via x="7.62" y="8.89" extent="1-16" drill="0.3"/>
 <via x="8.89" y="8.89" extent="1-16" drill="0.3"/>
@@
 <via x="16.51" y="19.05" extent="1-16" drill="0.3"/>
 <via x="8.89" y="13.97" extent="1-16" drill="0.3"/>
-<via x="7.62" y="17.78" extent="1-16" drill="0.3"/>
+<via x="6.35" y="19.05" extent="1-16" drill="0.3"/>
 <via x="15.24" y="17.145" extent="1-16" drill="0.3"/>
 </signal>
@@
 <wire x1="6.35" y1="13.208" x2="7.112" y2="13.208" width="0.6096" layer="16"/>
 <via x="7.112" y="13.208" extent="1-16" drill="0.3"/>
-<wire x1="7.112" y1="13.208" x2="6.731" y2="13.208" width="0.6096" layer="1"/>
-<wire x1="6.731" y1="13.208" x2="6.35" y2="13.208" width="0.6096" layer="1"/>
-<wire x1="6.77" y1="16.129" x2="6.77" y2="13.247" width="0.6096" layer="1"/>
-<wire x1="6.77" y1="13.247" x2="6.731" y2="13.208" width="0.6096" layer="1"/>
+<wire x1="7.112" y1="13.208" x2="6.35" y2="13.208" width="0.6096" layer="1"/>
+<wire x1="6.35" y1="13.208" x2="6.262" y2="13.296" width="0.6096" layer="1"/>
+<wire x1="6.262" y1="16.129" x2="6.262" y2="13.296" width="0.6096" layer="1"/>
 <wire x1="7.112" y1="13.208" x2="8.89" y2="11.43" width="0.6096" layer="16"/>
 <wire x1="8.89" y1="11.43" x2="24.13" y2="11.43" width="0.6096" layer="16"/>
+<contactref element="ILIM" pad="1"/>
+<wire x1="6.262" y1="16.129" x2="5.207" y2="16.129" width="0.6096" layer="1"/>
+<via x="5.207" y="16.129" extent="1-16" drill="0.3"/>
+<wire x1="5.207" y1="16.129" x2="6.7056" y2="16.129" width="0.6096" layer="16"/>
 </signal>
 <signal name="N$2">
@@
 <contactref element="FB1" pad="1"/>
 <contactref element="C3" pad="2"/>
-<wire x1="8.47" y1="16.129" x2="9.994" y2="16.129" width="0.6096" layer="1"/>
-<wire x1="9.994" y1="16.129" x2="10.033" y2="16.168" width="0.6096" layer="1"/>
 <wire x1="11.596" y1="16.129" x2="11.557" y2="16.168" width="0.6096" layer="1"/>
 <wire x1="11.557" y1="16.168" x2="10.033" y2="16.168" width="0.6096" layer="1"/>
+<contactref element="ILIM" pad="2"/>
+<wire x1="10.033" y1="16.168" x2="9.056" y2="16.168" width="0.6096" layer="1"/>
+<wire x1="9.056" y1="16.168" x2="9.017" y2="16.129" width="0.6096" layer="1"/>
+<via x="9.017" y="16.129" extent="1-16" drill="0.3"/>
+<wire x1="7.962" y1="16.129" x2="8.001" y2="16.168" width="0.6096" layer="1"/>
+<wire x1="8.001" y1="16.168" x2="9.056" y2="16.168" width="0.6096" layer="1"/>
+<wire x1="9.017" y1="16.129" x2="7.5184" y2="16.129" width="0.6096" layer="16"/>
 </signal>
 </signals>

Commit message: Ready for review
Parts:
- added LOGO3: SPECIAL_INSTRUCTIONS-ORDERING, SparkFun-Aesthetics:ORDERING_INSTRUCTIONS
- U$11: device output:#VIN#0 -> output:#VCC#0
- U$12: device output:#VIN#1 -> output:#VCC#1
- moved FRAME1 17.1 mm to (64.8, -10.2)
Connections:
- net N$4 renamed RF
- net VIN renamed VCC
Other:
- board text added: "2-layer PCB 1.6mm thickness 1oz Copper HASL lead-free surface finish Black solder resist White silkscreen"
- board text added: "Route Out"
- board text added: "x01"

Commit message: x01 PCB
Parts:
- U1: device BP2G1:XX21 -> SparkFun-RF:XX21
Routing:
- net GND: track 0.00 -> 1.85 mm, vias 69 -> 70
Changed lines of the file:
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@@
 <drawing>
 <settings>
-<setting alwaysvectorfont="no"/>
+<setting alwaysvectorfont="yes"/>
 <setting verticaltext="up"/>
 </settings>
@@
 <text x="12.7" y="0.381" size="1.27" layer="16" font="vector" ratio="15" rot="MR0" align="bottom-center">x01</text>
 <wire x1="12.446" y1="16.51" x2="12.446" y2="15.748" width="0.2032" layer="41"/>
+<wire x1="12.065" y1="6.35" x2="13.335" y2="6.35" width="0.2032" layer="41"/>
+<wire x1="8.636" y1="8.636" x2="8.636" y2="14.224" width="0.2032" layer="41"/>
+<wire x1="16.764" y1="8.636" x2="16.764" y2="14.986" width="0.2032" layer="41"/>
+<wire x1="15.24" y1="16.51" x2="16.764" y2="14.986" width="0.2032" layer="41"/>
+<wire x1="8.89" y1="7.239" x2="8.89" y2="6.477" width="0.2032" layer="41"/>
+<wire x1="16.51" y1="7.239" x2="16.51" y2="6.477" width="0.2032" layer="41"/>
 </plain>
 <attributes>
@@
 <attribute name="PROD_ID" value="CONN-08289" x="20.6375" y="4.7625" size="1.778" layer="27" ratio="15" rot="SR225" display="off"/>
 </element>
-<element name="U1" library="BP2G1" package="XX21" value="BP2G1+_POWER_SPLITTER" x="12.7" y="11.43" smashed="yes" rot="R180">
+<element name="U1" library="SparkFun-RF" package="XX21" value="BP2G1+_POWER_SPLITTER" x="12.7" y="11.43" smashed="yes" rot="R180">
 <attribute name="NAME" x="15.875" y="11.43" size="0.6096" layer="25" font="vector" ratio="20" rot="R270" align="bottom-center"/>
-<attribute name="PROD_ID" value="" x="12.7" y="11.43" size="1.778" layer="27" ratio="15" rot="R180" display="off"/>
+<attribute name="PROD_ID" value="IC-17198" x="12.7" y="11.43" size="1.778" layer="27" ratio="15" rot="R180" display="off"/>
 <attribute name="VALUE" x="8.89" y="11.43" size="0.6096" layer="27" font="vector" ratio="20" rot="R270" align="bottom-center"/>
 </element>
@@
 <contactref element="D1" pad="2"/>
 <contactref element="C3" pad="1"/>
-<polygon width="0.3048" layer="1" isolate="0.2032">
+<polygon width="0.6096" layer="1" isolate="0.2032">
 <vertex x="0" y="25.4"/>
 <vertex x="25.4" y="25.4"/>
@@
 <vertex x="0" y="0"/>
 </polygon>
-<via x="10.795" y="13.081" extent="1-16" drill="0.3"/>
-<via x="12.065" y="13.081" extent="1-16" drill="0.3"/>
-<via x="14.605" y="13.081" extent="1-16" drill="0.3"/>
-<via x="9.906" y="14.732" extent="1-16" drill="0.3"/>
+<via x="10.795" y="12.827" extent="1-16" drill="0.3"/>
+<via x="12.065" y="12.827" extent="1-16" drill="0.3"/>
+<via x="14.605" y="12.827" extent="1-16" drill="0.3"/>
+<via x="9.525" y="14.224" extent="1-16" drill="0.3"/>
 <via x="7.62" y="14.732" extent="1-16" drill="0.3"/>
 <via x="5.08" y="15.24" extent="1-16" drill="0.3"/>
@@
 <via x="14.605" y="10.033" extent="1-16" drill="0.3"/>
 <via x="10.795" y="10.033" extent="1-16" drill="0.3"/>
-<via x="13.335" y="13.081" extent="1-16" drill="0.3"/>
+<via x="13.335" y="12.827" extent="1-16" drill="0.3"/>
 <via x="11.557" y="18.542" extent="1-16" drill="0.3"/>
 <via x="15.24" y="18.542" extent="1-16" drill="0.3"/>
-<via x="8.89" y="19.05" extent="1-16" drill="0.3"/>
+<via x="8.89" y="18.796" extent="1-16" drill="0.3"/>
 <via x="8.382" y="20.32" extent="1-16" drill="0.3"/>
 <via x="8.382" y="23.368" extent="1-16" drill="0.3"/>
@@
 <via x="17.018" y="21.844" extent="1-16" drill="0.3"/>
 <via x="17.018" y="20.32" extent="1-16" drill="0.3"/>
-<via x="14.605" y="16.129" extent="1-16" drill="0.3"/>
+<via x="14.605" y="15.367" extent="1-16" drill="0.3"/>
 <via x="12.065" y="7.366" extent="1-16" drill="0.3"/>
 <via x="13.335" y="7.366" extent="1-16" drill="0.3"/>
@@
 <via x="6.35" y="10.16" extent="1-16" drill="0.3"/>
 <via x="7.62" y="10.16" extent="1-16" drill="0.3"/>
-<via x="16.51" y="10.16" extent="1-16" drill="0.3"/>
-<via x="8.89" y="10.16" extent="1-16" drill="0.3"/>
+<via x="15.875" y="10.033" extent="1-16" drill="0.3"/>
+<via x="9.525" y="10.033" extent="1-16" drill="0.3"/>
 <via x="17.78" y="10.16" extent="1-16" drill="0.3"/>
 <via x="19.05" y="10.16" extent="1-16" drill="0.3"/>
 <via x="20.32" y="10.16" extent="1-16" drill="0.3"/>
-<via x="16.51" y="12.7" extent="1-16" drill="0.3"/>
+<via x="15.875" y="12.827" extent="1-16" drill="0.3"/>
 <via x="17.78" y="12.7" extent="1-16" drill="0.3"/>
 <via x="19.05" y="12.7" extent="1-16" drill="0.3"/>
@@
 <via x="21.59" y="10.16" extent="1-16" drill="0.3"/>
 <via x="3.81" y="11.43" extent="1-16" drill="0.3"/>
-<via x="7.62" y="8.89" extent="1-16" drill="0.3"/>
-<via x="8.89" y="8.89" extent="1-16" drill="0.3"/>
+<via x="7.62" y="8.636" extent="1-16" drill="0.3"/>
+<via x="9.525" y="8.636" extent="1-16" drill="0.3"/>
 <via x="10.16" y="5.08" extent="1-16" drill="0.3"/>
 <via x="11.43" y="5.08" extent="1-16" drill="0.3"/>
@@
 <via x="13.97" y="5.08" extent="1-16" drill="0.3"/>
 <via x="15.24" y="5.08" extent="1-16" drill="0.3"/>
-<via x="16.51" y="8.89" extent="1-16" drill="0.3"/>
-<via x="17.78" y="8.89" extent="1-16" drill="0.3"/>
+<via x="15.875" y="8.636" extent="1-16" drill="0.3"/>
+<via x="17.78" y="8.636" extent="1-16" drill="0.3"/>
 <via x="19.05" y="8.89" extent="1-16" drill="0.3"/>
 <via x="20.32" y="8.89" extent="1-16" drill="0.3"/>
 <via x="5.08" y="8.89" extent="1-16" drill="0.3"/>
-<via x="16.51" y="15.24" extent="1-16" drill="0.3"/>
+<via x="15.875" y="14.224" extent="1-16" drill="0.3"/>
 <via x="16.51" y="19.05" extent="1-16" drill="0.3"/>
-<via x="8.89" y="13.97" extent="1-16" drill="0.3"/>
+<via x="9.525" y="12.827" extent="1-16" drill="0.3"/>
 <via x="6.35" y="19.05" extent="1-16" drill="0.3"/>
-<via x="15.24" y="17.145" extent="1-16" drill="0.3"/>
+<via x="14.605" y="17.145" extent="1-16" drill="0.3"/>
 <polygon width="0.3048" layer="1" isolate="0.127" rank="2">
-<vertex x="0" y="10.16"/>
-<vertex x="25.4" y="10.16"/>
-<vertex x="25.4" y="0"/>
-<vertex x="0" y="0"/>
+<vertex x="10.795" y="25.4"/>
+<vertex x="14.605" y="25.4"/>
+<vertex x="14.605" y="16.764"/>
+<vertex x="14.323540625" y="16.482540625"/>
+<vertex x="14.224" y="12.7"/>
+<vertex x="12.446" y="12.7"/>
+<vertex x="12.446" y="16.51"/>
+<vertex x="10.795" y="18.161"/>
 </polygon>
 <polygon width="0.3048" layer="1" isolate="0.127" rank="2">
-<vertex x="11.176" y="25.4"/>
-<vertex x="14.605" y="25.4"/>
-<vertex x="14.605" y="12.7"/>
-<vertex x="11.176" y="12.7"/>
+<vertex x="1.7145" y="4.6355"/>
+<vertex x="4.6355" y="1.7145"/>
+<vertex x="8.001" y="5.08"/>
+<vertex x="17.399" y="5.08"/>
+<vertex x="20.7645" y="1.7145"/>
+<vertex x="23.6855" y="4.6355"/>
+<vertex x="20.447" y="7.874"/>
+<vertex x="15.875" y="7.874"/>
+<vertex x="15.875" y="10.033"/>
+<vertex x="9.525" y="10.033"/>
+<vertex x="9.525" y="7.874"/>
+<vertex x="4.953" y="7.874"/>
 </polygon>
+<wire x1="13.589" y1="18.542" x2="13.589" y2="19.304" width="0.508" layer="1"/>
+<wire x1="13.915" y1="18.542" x2="13.589" y2="18.542" width="0.3048" layer="1"/>
+<wire x1="13.589" y1="18.542" x2="13.589" y2="17.78" width="0.508" layer="1"/>
+<via x="11.557" y="17.526" extent="1-16" drill="0.3"/>
 </signal>
 <signal name="RF">
