File: Hardware/Production/GNSS_Splitter-Panel.brd (EAGLE design)
At the start: 175 x 117.3 mm, 1014 parts, among them J1 QWIIC_RIGHT_ANGLE, J11 QWIIC_RIGHT_ANGLE, J13 QWIIC_RIGHT_ANGLE, J15 QWIIC_RIGHT_ANGLE, J17 QWIIC_RIGHT_ANGLE, J19 QWIIC_RIGHT_ANGLE, J21 QWIIC_RIGHT_ANGLE, J23 QWIIC_RIGHT_ANGLE, J25 QWIIC_RIGHT_ANGLE, J27 QWIIC_RIGHT_ANGLE, J29 QWIIC_RIGHT_ANGLE, J3 QWIIC_RIGHT_ANGLE, J31 QWIIC_RIGHT_ANGLE, J33 QWIIC_RIGHT_ANGLE, J35 QWIIC_RIGHT_ANGLE, J37 QWIIC_RIGHT_ANGLE, J39 QWIIC_RIGHT_ANGLE, J41 QWIIC_RIGHT_ANGLE, J43 QWIIC_RIGHT_ANGLE, J45 QWIIC_RIGHT_ANGLE, J47 QWIIC_RIGHT_ANGLE, J5 QWIIC_RIGHT_ANGLE, J7 QWIIC_RIGHT_ANGLE, J9 QWIIC_RIGHT_ANGLE, U1 BP2G1+_POWER_SPLITTER, U10 BP2G1+_POWER_SPLITTER, U11 BP2G1+_POWER_SPLITTER, U12 BP2G1+_POWER_SPLITTER, U13 BP2G1+_POWER_SPLITTER, U14 BP2G1+_POWER_SPLITTER, U15 BP2G1+_POWER_SPLITTER, U16 BP2G1+_POWER_SPLITTER, U17 BP2G1+_POWER_SPLITTER, U18 BP2G1+_POWER_SPLITTER, U19 BP2G1+_POWER_SPLITTER, U2 BP2G1+_POWER_SPLITTER, U20 BP2G1+_POWER_SPLITTER, U21 BP2G1+_POWER_SPLITTER, U22 BP2G1+_POWER_SPLITTER, U23 BP2G1+_POWER_SPLITTER, U24 BP2G1+_POWER_SPLITTER, U3 BP2G1+_POWER_SPLITTER, U4 BP2G1+_POWER_SPLITTER, U5 BP2G1+_POWER_SPLITTER, U6 BP2G1+_POWER_SPLITTER, U7 BP2G1+_POWER_SPLITTER, U8 BP2G1+_POWER_SPLITTER, U9 BP2G1+_POWER_SPLITTER

Commit message: x01 PCB
Parts:
- U1, U10, U11, U12, U13, U14, U15, U16, U17, U18, U19, U2, U20, U21, U22, U23, U24, U3, U4, U5, U6, U7, U8, U9: device BP2G1:XX21 -> SparkFun-RF:XX21
Routing:
- net GND23: track 0.00 -> 1.85 mm, vias 69 -> 70
- net GND17: track 0.00 -> 1.85 mm, vias 69 -> 70
- net GND11: track 0.00 -> 1.85 mm, vias 69 -> 70
- net GND5: track 0.00 -> 1.85 mm, vias 69 -> 70
- net GND7: track 0.00 -> 1.85 mm, vias 69 -> 70
- net GND19: track 0.00 -> 1.85 mm, vias 69 -> 70
- net GND13: track 0.00 -> 1.85 mm, vias 69 -> 70
- net GND6: track 0.00 -> 1.85 mm, vias 69 -> 70
- net GND18: track 0.00 -> 1.85 mm, vias 69 -> 70
- net GND12: track 0.00 -> 1.85 mm, vias 69 -> 70
- net GND1: track 0.00 -> 1.85 mm, vias 69 -> 70
- net GND: track 0.00 -> 1.85 mm, vias 69 -> 70
- net GND9: track 0.00 -> 1.85 mm, vias 69 -> 70
- net GND8: track 0.00 -> 1.85 mm, vias 69 -> 70
- net GND22: track 0.00 -> 1.85 mm, vias 69 -> 70
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